File: hardware/kitchen_timer_6.4/kitchen_timer_6.4.kicad_pcb (KiCad board)
At the start: 2 copper layers, 79.5 x 66 mm, 55 parts, among them J1 USB_C, J2 BREAKOUT, J3 JST PH 2.0, Q1 MMBT2222A, Q2 MMBT2222A, Q3 MMBT2222A, Q4 MMBT2222A, Q5 MMBT2222A, SW1 VOLUME, SW2 FUNCTION_SELECTOR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

Commit message: extra capacitor
Parts:
- added C4: 10u, 00_local:C_0805_2012Metric_Pad1.18x1.45mm_HandSolder, F.Cu at (112.2, 44.7)
- renumbered C4 to C1, C5 to C2, C1 to C3, C2 to C5, C3 to C6, D3 to D2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
Routing:
- net GND: track 32.0 -> 33.2 mm, vias 89 -> 87
