File: hardware/kitchen_timer_6.4/kitchen_timer_6.4.kicad_pcb (KiCad board)
At the start: 2 copper layers, 79.5 x 66 mm, 56 parts, among them J1 JST PH 2.0, J2 USB_C, J3 BREAKOUT, Q1 MMBT2222A, Q2 MMBT2222A, Q3 MMBT2222A, Q4 MMBT2222A, Q5 MMBT2222A, SW1 ON/OFF, SW2 SECONDS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

Commit message: redid the schematic without reannotating.  Hoping to me the usb -> battery charger -> boost converter more clear
Parts:
- C4: value 10u -> 22u
- R19: value 1R -> 5R
Connections:
- net +V_USB renamed /VBUS
- net A renamed /A
- net B renamed /B
- net BAT+ renamed /BAT+
- net BAT_LEVEL renamed /BAT_LEVEL
- net BAT_SW renamed /BAT_SW
- net BUZZER renamed /BUZZER
- net C renamed /C
- net CC1 renamed /CC1
- net CC2 renamed /CC2
- net CC3 renamed /CC3
- net CC4 renamed /CC4
- net D renamed /D
- net DIGIT_1 renamed /DIGIT_1
- net DIGIT_2 renamed /DIGIT_2
- net DIGIT_3 renamed /DIGIT_3
- net DIGIT_4 renamed /DIGIT_4
- net DP renamed /DP
- net E renamed /E
- net F renamed /F
- net FUNCTION renamed /FUNCTION
- net G renamed /G
- net MINUTES renamed /MINUTES
- net RESET_TIME renamed /RESET_TIME
- net RXD renamed /RXD
- net SECONDS renamed /SECONDS
- net START_STOP renamed /START_STOP
- net TEMP_GND renamed /TEMP_GND
- net TEMP_V renamed /TEMP_V
- net TXD renamed /TXD
- net UPDI renamed /UPDI
